Commit message: feat: completely isolate left/right hand retargeting pipelines, fix finger abduction, amplify thumb elevation, and sync left URDF joint01 axis with HW

File: urdf/allegro_hand_v6_left.urdf (robot description, URDF)
Before this commit: robot allegro_hand_v6_left, 21 links, 20 joints
Joints:
- joint joint01: axis 0 0 -1 -> 0 0 1

Commit message: fix: invert left thumb joint01 axis to match real HW, apply -90 deg motor offset to index-pinky joint1 and expand lower limits

File: urdf/allegro_hand_v6_left.urdf (robot description, URDF)
Before this commit: robot allegro_hand_v6_left, 21 links, 20 joints
Joints:
- joint joint01: axis 0 0 1 -> 0 0 -1
- joint joint11: limit lower=-0.0698132 upper=1.5707963 effort=15.0 velocity=7.0 -> lower=-1.6580628 upper=1.5707963 effort=15.0 velocity=7.0
- joint joint21: limit lower=-0.0698132 upper=1.5707963 effort=15.0 velocity=7.0 -> lower=-1.6580628 upper=1.5707963 effort=15.0 velocity=7.0
- joint joint31: limit lower=-0.0698132 upper=1.5707963 effort=15.0 velocity=7.0 -> lower=-1.6580628 upper=1.5707963 effort=15.0 velocity=7.0
- joint joint41: limit lower=-0.0698132 upper=1.5707963 effort=15.0 velocity=7.0 -> lower=-1.6580628 upper=1.5707963 effort=15.0 velocity=7.0

Commit message: fix: restore joint11-41 motor zero position at 0.0 rad to prevent curling, keep joint01 negative axis

File: urdf/allegro_hand_v6_left.urdf (robot description, URDF)
Before this commit: robot allegro_hand_v6_left, 21 links, 20 joints
Joints:
- joint joint11: limit lower=-1.6580628 upper=1.5707963 effort=15.0 velocity=7.0 -> lower=-0.0698132 upper=1.5707963 effort=15.0 velocity=7.0
- joint joint21: limit lower=-1.6580628 upper=1.5707963 effort=15.0 velocity=7.0 -> lower=-0.0698132 upper=1.5707963 effort=15.0 velocity=7.0
- joint joint31: limit lower=-1.6580628 upper=1.5707963 effort=15.0 velocity=7.0 -> lower=-0.0698132 upper=1.5707963 effort=15.0 velocity=7.0
- joint joint41: limit lower=-1.6580628 upper=1.5707963 effort=15.0 velocity=7.0 -> lower=-0.0698132 upper=1.5707963 effort=15.0 velocity=7.0

Commit message: fix: apply -90 deg motor offset to index-pinky joint 1, expand limits, and resolve socket linger and script paths

File: urdf/allegro_hand_v6_left.urdf (robot description, URDF)
Before this commit: robot allegro_hand_v6_left, 21 links, 20 joints
Joints:
- joint joint11: limit lower=-0.0698132 upper=1.5707963 effort=15.0 velocity=7.0 -> lower=-1.6580628 upper=1.5707963 effort=15.0 velocity=7.0
- joint joint21: limit lower=-0.0698132 upper=1.5707963 effort=15.0 velocity=7.0 -> lower=-1.6580628 upper=1.5707963 effort=15.0 velocity=7.0
- joint joint31: limit lower=-0.0698132 upper=1.5707963 effort=15.0 velocity=7.0 -> lower=-1.6580628 upper=1.5707963 effort=15.0 velocity=7.0
- joint joint41: limit lower=-0.0698132 upper=1.5707963 effort=15.0 velocity=7.0 -> lower=-1.6580628 upper=1.5707963 effort=15.0 velocity=7.0

Commit message: fix: normalize left thumb URDF opposition sign to prevent backwards bending and harden modbus IP auto-discovery

File: urdf/allegro_hand_v6_left.urdf (robot description, URDF)
Before this commit: robot allegro_hand_v6_left, 21 links, 20 joints
Joints:
- joint joint00: limit lower=-1.6580628 upper=1.6580628 effort=15.0 velocity=7.0 -> lower=-0.0349066 upper=1.6580628 effort=15.0 velocity=7.0

Commit message: fix(kinematics): decouple real left hand motor offset from URDF, add startup zero position, and isolate abduction from MCP flexion

File: urdf/allegro_hand_v6_left.urdf (robot description, URDF)
Before this commit: robot allegro_hand_v6_left, 21 links, 20 joints
Joints:
- joint joint11: limit lower=-0.0698132 upper=1.5707963 effort=15.0 velocity=7.0 -> lower=-1.6580628 upper=1.5707963 effort=15.0 velocity=7.0
- joint joint21: limit lower=-0.0698132 upper=1.5707963 effort=15.0 velocity=7.0 -> lower=-1.6580628 upper=1.5707963 effort=15.0 velocity=7.0
- joint joint31: limit lower=-0.0698132 upper=1.5707963 effort=15.0 velocity=7.0 -> lower=-1.6580628 upper=1.5707963 effort=15.0 velocity=7.0
- joint joint41: limit lower=-0.0698132 upper=1.5707963 effort=15.0 velocity=7.0 -> lower=-1.6580628 upper=1.5707963 effort=15.0 velocity=7.0

File: urdf/allegro_hand_v6_left_v6.1_teleop.urdf (robot description, URDF)
Before this commit: robot allegro_hand_v6_left, 21 links, 20 joints
Joints:
- joint joint00: limit lower=-1.6580628 upper=1.6580628 effort=15.0 velocity=7.0 -> lower=-0.0349066 upper=1.6580628 effort=15.0 velocity=7.0
