Commit message: urdf: take the driver's own left and right URDFs
The repo keeps a copy of the driver URDF for the cockpit's 3D view. The left copy
had drifted: joint10/20/30/40 carried the opposite axis sign with the limits negated
and swapped, which is the same geometry described with the opposite joint sign, so
the cockpit drew the left hand's abduction mirrored against the joint values the
driver reports. Both copies now come from the driver package unchanged.

Note in the README that the left hand reads its meshes from meshes/left/, which has
to exist in the driver sources, and that these copies track the driver package.

Co-Authored-By: Claude Opus 5 <noreply@anthropic.com>

File: urdf/allegro_hand_v6_left.urdf (robot description, URDF)
Before this commit: robot allegro_hand_v6_left, 21 links, 20 joints
Joints:
- joint joint10: axis 0 0 -1 -> 0 0 1; limit lower=-0.3839724 upper=1.3089969 effort=15.0 velocity=7.0 -> lower=-1.3089969 upper=0.3839724 effort=15.0 velocity=7.0
- joint joint20: axis 0 0 -1 -> 0 0 1
- joint joint30: axis 0 0 -1 -> 0 0 1; limit lower=-1.3089969 upper=0.3839724 effort=15.0 velocity=7.0 -> lower=-0.3839724 upper=1.3089969 effort=15.0 velocity=7.0
- joint joint40: axis 0 0 -1 -> 0 0 1; limit lower=-1.3089969 upper=0.4363323 effort=15.0 velocity=7.0 -> lower=-0.4363323 upper=1.3089969 effort=15.0 velocity=7.0

Commit message: urdf: keep the left abduction signs the hardware actually reports
The previous commit took the driver package's left URDF wholesale. Measuring the
hand says that was wrong for four joints. Spreading each finger by hand and reading
the encoders (no commands sent) gives index joint10 a range of -0.40 to +1.39 rad and
ring joint30 -1.28 to +0.41, where the driver's URDF allows +0.38 and -0.38 in those
directions. This left hand signs its abduction the way the right hand does, which is
what the MANUS teleop project's URDF already described, and the driver package's
mirrored description does not match it.

So joint10/20/30/40 keep axis "0 0 -1" with the limits negated and swapped, and the
file and the README now say why, with the measurement, so that the next driver update
does not quietly undo it. The left hand runs firmware 0x0103 against the right hand's
0x0300, which is worth raising with Wonik.

Everything else, both hands, stays the driver package's own.

Co-Authored-By: Claude Opus 5 <noreply@anthropic.com>

File: urdf/allegro_hand_v6_left.urdf (robot description, URDF)
Before this commit: robot allegro_hand_v6_left, 21 links, 20 joints
Joints:
- joint joint10: axis 0 0 1 -> 0 0 -1; limit lower=-1.3089969 upper=0.3839724 effort=15.0 velocity=7.0 -> lower=-0.3839724 upper=1.3089969 effort=15.0 velocity=7.0
- joint joint20: axis 0 0 1 -> 0 0 -1
- joint joint30: axis 0 0 1 -> 0 0 -1; limit lower=-0.3839724 upper=1.3089969 effort=15.0 velocity=7.0 -> lower=-1.3089969 upper=0.3839724 effort=15.0 velocity=7.0
- joint joint40: axis 0 0 1 -> 0 0 -1; limit lower=-0.4363323 upper=1.3089969 effort=15.0 velocity=7.0 -> lower=-1.3089969 upper=0.4363323 effort=15.0 velocity=7.0
