Commit message: Make the ROS 2 Jazzy version the repository root; freeze Humble under humble/
- Jazzy (native, Ubuntu 24.04) files move from jazzy/ to the root: it is the main line,
  with v3 = DexPilot retargeting, tactile pressure panel, smoothed input, hand discovery
- The ROS 2 Humble + docker version moves to humble/ and is frozen; its launchers
  re-execute inside the container, so their fixed paths now point at .../humble/
- README: full environment setup (ROS 2 Jazzy, Wonik driver workspace, DexPilot core
  and its venv, this repo, network) and the Humble/Jazzy differences
- run_dashboard.sh always runs the latest pipeline (v3, with the tactile panel);
  --v2 / --v1 select the earlier ones
- Hand discovery prefers HAND_SIDE (right by default) when both hands are connected

Co-Authored-By: Claude Opus 5.5 <noreply@anthropic.com>

File: humble/urdf/allegro_hand_v6_left_v6.1_teleop.urdf (robot description, URDF)
Before this commit: robot allegro_hand_v6_left, 21 links, 20 joints
Joints:
- joint joint10: axis 0 0 -1 -> 0 0 1; limit lower=-0.3839724 upper=1.3089969 effort=15.0 velocity=7.0 -> lower=-1.3089969 upper=0.3839724 effort=15.0 velocity=7.0
- joint joint11: limit lower=-0.0698132 upper=1.5707963 effort=15.0 velocity=7.0 -> lower=-1.6580628 upper=1.5707963 effort=15.0 velocity=7.0
- joint joint20: axis 0 0 -1 -> 0 0 1
- joint joint21: limit lower=-0.0698132 upper=1.5707963 effort=15.0 velocity=7.0 -> lower=-1.6580628 upper=1.5707963 effort=15.0 velocity=7.0
- joint joint30: axis 0 0 -1 -> 0 0 1; limit lower=-1.3089969 upper=0.3839724 effort=15.0 velocity=7.0 -> lower=-0.3839724 upper=1.3089969 effort=15.0 velocity=7.0
- joint joint31: limit lower=-0.0698132 upper=1.5707963 effort=15.0 velocity=7.0 -> lower=-1.6580628 upper=1.5707963 effort=15.0 velocity=7.0
- joint joint40: axis 0 0 -1 -> 0 0 1; limit lower=-1.3089969 upper=0.4363323 effort=15.0 velocity=7.0 -> lower=-0.4363323 upper=1.3089969 effort=15.0 velocity=7.0
- joint joint41: limit lower=-0.0698132 upper=1.5707963 effort=15.0 velocity=7.0 -> lower=-1.6580628 upper=1.5707963 effort=15.0 velocity=7.0
